File: WeatherStation_PCB/weatherstation.sch (EAGLE design)
At the start: 17 parts

Commit message: Fixed Issue #3 Updated the design to contain the 5V jumper.
Parts:
- added 5V_JUMP: (no value), rcl:R-US_R0805
Connections:
- new net N$3: 5V_JUMP.1, U$1.5V
- net 5V: now also 5V_JUMP.2; no longer U$1.5V
Changed lines of the file:
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@@
 <part name="3P3V_JUMP" library="rcl" deviceset="R-US_" device="R0805"/>
 <part name="5_REG" library="SparkFun-PowerIC" deviceset="V_REG_MIC2920" device=""/>
+<part name="5V_JUMP" library="rcl" deviceset="R-US_" device="R0805"/>
 </parts>
 <sheets>
@@
 <instance part="C4" gate="G$1" x="165.1" y="73.66"/>
 <instance part="3P3_REG" gate="G$1" x="121.92" y="106.68"/>
-<instance part="3P3V_JUMP" gate="G$1" x="53.34" y="53.34" rot="R180"/>
+<instance part="3P3V_JUMP" gate="G$1" x="53.34" y="53.34" smashed="yes" rot="R180">
+<attribute name="NAME" x="61.214" y="55.1434" size="1.778" layer="95" rot="R180"/>
+<attribute name="VALUE" x="57.15" y="56.642" size="1.778" layer="96" rot="R180"/>
+</instance>
 <instance part="5_REG" gate="G$1" x="157.48" y="106.68"/>
+<instance part="5V_JUMP" gate="G$1" x="53.34" y="55.88" smashed="yes" rot="R180">
+<attribute name="NAME" x="59.182" y="57.6834" size="1.778" layer="95" rot="R180"/>
+<attribute name="VALUE" x="57.15" y="59.182" size="1.778" layer="96" rot="R180"/>
+</instance>
 </instances>
 <busses>
@@
 </segment>
 <segment>
-<pinref part="U$1" gate="G$1" pin="5V"/>
-<wire x1="63.5" y1="55.88" x2="43.18" y2="55.88" width="0.1524" layer="91"/>
-<label x="50.8" y="55.88" size="1.778" layer="95"/>
-</segment>
-<segment>
 <pinref part="3P3_REG" gate="G$1" pin="IN"/>
 <wire x1="114.3" y1="106.68" x2="111.76" y2="106.68" width="0.1524" layer="91"/>
@@
 <label x="167.64" y="106.68" size="1.778" layer="95"/>
 </segment>
+<segment>
+<pinref part="5V_JUMP" gate="G$1" pin="2"/>
+<wire x1="48.26" y1="55.88" x2="43.18" y2="55.88" width="0.1524" layer="91"/>
+</segment>
 </net>
 <net name="MOSI" class="0">
@@
 </segment>
 </net>
+<net name="N$3" class="0">
+<segment>
+<pinref part="U$1" gate="G$1" pin="5V"/>
+<pinref part="5V_JUMP" gate="G$1" pin="1"/>
+<wire x1="63.5" y1="55.88" x2="58.42" y2="55.88" width="0.1524" layer="91"/>
+</segment>
+</net>
